Commit message: test new urdf_aliengo

File: motion_imitation/utilities/aliengo_description/urdf/aliengo.urdf (robot description, URDF)
Before this commit: robot aliengo_description, 18 links, 17 joints
Links:
- added link FL_calf_rotor, mass 0.132; collision cylinder length=0.02 radius=0.035; visual cylinder length=0.02 radius=0.035
- added link FL_hip_rotor, mass 0.146; collision cylinder length=0.02 radius=0.035; visual cylinder length=0.02 radius=0.035
- added link FL_thigh_rotor, mass 0.146; collision cylinder length=0.02 radius=0.035; visual cylinder length=0.02 radius=0.035
- added link FR_calf_rotor, mass 0.132; collision cylinder length=0.02 radius=0.035; visual cylinder length=0.02 radius=0.035
- added link FR_hip_rotor, mass 0.146; collision cylinder length=0.02 radius=0.035; visual cylinder length=0.02 radius=0.035
- added link FR_thigh_rotor, mass 0.146; collision cylinder length=0.02 radius=0.035; visual cylinder length=0.02 radius=0.035
- added link RL_calf_rotor, mass 0.132; collision cylinder length=0.02 radius=0.035; visual cylinder length=0.02 radius=0.035
- added link RL_hip_rotor, mass 0.146; collision cylinder length=0.02 radius=0.035; visual cylinder length=0.02 radius=0.035
- added link RL_thigh_rotor, mass 0.146; collision cylinder length=0.02 radius=0.035; visual cylinder length=0.02 radius=0.035
- added link RR_calf_rotor, mass 0.132; collision cylinder length=0.02 radius=0.035; visual cylinder length=0.02 radius=0.035
- added link RR_hip_rotor, mass 0.146; collision cylinder length=0.02 radius=0.035; visual cylinder length=0.02 radius=0.035
- added link RR_thigh_rotor, mass 0.146; collision cylinder length=0.02 radius=0.035; visual cylinder length=0.02 radius=0.035
- link FL_calf: geometry collision box size=0.25 0.0208 0.016; visual mesh filename=package://aliengo_description/meshes/calf.dae scale=1 1 1
- link FL_hip: geometry collision cylinder length=0.0418 radius=0.046; visual mesh filename=package://aliengo_description/meshes/hip.dae scale=1 1 1
- link FL_thigh: geometry collision box size=0.25 0.0374 0.043; visual mesh filename=package://aliengo_description/meshes/thigh.dae scale=1 1 1
- link FR_calf: geometry collision box size=0.25 0.0208 0.016; visual mesh filename=package://aliengo_description/meshes/calf.dae scale=1 1 1
- link FR_hip: geometry collision cylinder length=0.0418 radius=0.046; visual mesh filename=package://aliengo_description/meshes/hip.dae scale=1 1 1
- link FR_thigh: geometry collision box size=0.25 0.0374 0.043; visual mesh filename=package://aliengo_description/meshes/thigh_mirror.dae scale=1 1 1
- link RL_calf: geometry collision box size=0.25 0.0208 0.016; visual mesh filename=package://aliengo_description/meshes/calf.dae scale=1 1 1
- link RL_hip: geometry collision cylinder length=0.0418 radius=0.046; visual mesh filename=package://aliengo_description/meshes/hip.dae scale=1 1 1
- link RL_thigh: geometry collision box size=0.25 0.0374 0.043; visual mesh filename=package://aliengo_description/meshes/thigh.dae scale=1 1 1
- link RR_calf: geometry collision box size=0.25 0.0208 0.016; visual mesh filename=package://aliengo_description/meshes/calf.dae scale=1 1 1
- link RR_hip: geometry collision cylinder length=0.0418 radius=0.046; visual mesh filename=package://aliengo_description/meshes/hip.dae scale=1 1 1
- link RR_thigh: geometry collision box size=0.25 0.0374 0.043; visual mesh filename=package://aliengo_description/meshes/thigh_mirror.dae scale=1 1 1
- link trunk: mass 9.041 -> 11.644; geometry collision box size=0.647 0.15 0.112; visual mesh filename=package://aliengo_description/meshes/trunk.dae scale=1 1 1
Joints:
- removed joint RR_toe_fixed
- added joint FL_calf_rotor_joint: type fixed, parent FL_thigh, child FL_calf_rotor, origin xyz=0.0 -0.0997 0 rpy=0 0 0
- added joint FL_hip_rotor_joint: type fixed, parent trunk, child FL_hip_rotor, origin xyz=0.139985 0.051 0 rpy=0 0 0
- added joint FL_thigh_rotor_joint: type fixed, parent FL_hip, child FL_thigh_rotor, origin xyz=0.0 0.0298 0 rpy=0 0 0
- added joint FR_calf_rotor_joint: type fixed, parent FR_thigh, child FR_calf_rotor, origin xyz=0.0 0.0997 0 rpy=0 0 0
- added joint FR_thigh_rotor_joint: type fixed, parent FR_hip, child FR_thigh_rotor, origin xyz=0.0 -0.0298 0 rpy=0 0 0
- added joint RL_calf_rotor_joint: type fixed, parent RL_thigh, child RL_calf_rotor, origin xyz=0.0 -0.0997 0 rpy=0 0 0
- added joint RL_hip_rotor_joint: type fixed, parent trunk, child RL_hip_rotor, origin xyz=-0.139985 0.051 0 rpy=0 0 0
- added joint RL_thigh_rotor_joint: type fixed, parent RL_hip, child RL_thigh_rotor, origin xyz=0.0 0.0298 0 rpy=0 0 0
- added joint RR_calf_rotor_joint: type fixed, parent RR_thigh, child RR_calf_rotor, origin xyz=0.0 0.0997 0 rpy=0 0 0
- added joint RR_foot_fixed: type fixed, parent RR_calf, child RR_foot, origin xyz=0 0 -0.25 rpy=0 0 0
- added joint RR_hip_rotor_joint: type fixed, parent trunk, child RR_hip_rotor, origin xyz=-0.139985 -0.051 0 rpy=0 0 0
- added joint RR_thigh_rotor_joint: type fixed, parent RR_hip, child RR_thigh_rotor, origin xyz=0.0 -0.0298 0 rpy=0 0 0
- joint FL_calf_joint: limit lower=-2.77507351067 upper=-0.645771823238 effort=44.4 velocity=40 -> lower=-2.775073510670984 upper=-0.6457718232379019 effort=44.4 velocity=15.89
- joint FL_hip_joint: limit lower=-1.2217304764 upper=1.2217304764 effort=44.4 velocity=40 -> lower=-1.2217304763960306 upper=1.2217304763960306 effort=35.278 velocity=20; origin xyz=0.2399 0.051 0 rpy=0 0 0 -> xyz=0.2407 0.051 0 rpy=0 0 0
- joint FL_thigh_joint: limit effort=44.4 velocity=40 -> effort=35.278 velocity=20; origin xyz=0 0.083 0 rpy=0 0 0 -> xyz=0 0.0868 0 rpy=0 0 0
- joint FL_toe_fixed: child FL_toe -> FL_foot
- joint FR_calf_joint: limit lower=-2.77507351067 upper=-0.645771823238 effort=44.4 velocity=40 -> lower=-2.775073510670984 upper=-0.6457718232379019 effort=44.4 velocity=15.89
- joint FR_hip_joint: limit lower=-1.2217304764 upper=1.2217304764 effort=44.4 velocity=40 -> lower=-1.2217304763960306 upper=1.2217304763960306 effort=35.278 velocity=20; origin xyz=0.2399 -0.051 0 rpy=0 0 0 -> xyz=0.2407 -0.051 0 rpy=0 0 0
- joint FR_thigh_joint: limit effort=44.4 velocity=40 -> effort=35.278 velocity=20; origin xyz=0 -0.083 0 rpy=0 0 0 -> xyz=0 -0.0868 0 rpy=0 0 0
- joint FR_toe_fixed: child FR_toe -> FR_foot
- joint RL_calf_joint: limit lower=-2.77507351067 upper=-0.645771823238 effort=44.4 velocity=40 -> lower=-2.775073510670984 upper=-0.6457718232379019 effort=44.4 velocity=15.89
- joint RL_hip_joint: limit lower=-1.2217304764 upper=1.2217304764 effort=44.4 velocity=40 -> lower=-1.2217304763960306 upper=1.2217304763960306 effort=35.278 velocity=20; origin xyz=-0.2399 0.051 0 rpy=0 0 0 -> xyz=-0.2407 0.051 0 rpy=0 0 0
- joint RL_thigh_joint: limit effort=44.4 velocity=40 -> effort=35.278 velocity=20; origin xyz=0 0.083 0 rpy=0 0 0 -> xyz=0 0.0868 0 rpy=0 0 0
- joint RL_toe_fixed: child RL_toe -> RL_foot
- joint RR_calf_joint: limit lower=-2.77507351067 upper=-0.645771823238 effort=44.4 velocity=40 -> lower=-2.775073510670984 upper=-0.6457718232379019 effort=44.4 velocity=15.89
- joint RR_hip_joint: limit lower=-1.2217304764 upper=1.2217304764 effort=44.4 velocity=40 -> lower=-1.2217304763960306 upper=1.2217304763960306 effort=35.278 velocity=20; origin xyz=-0.2399 -0.051 0 rpy=0 0 0 -> xyz=-0.2407 -0.051 0 rpy=0 0 0
- joint RR_thigh_joint: limit effort=44.4 velocity=40 -> effort=35.278 velocity=20; origin xyz=0 -0.083 0 rpy=0 0 0 -> xyz=0 -0.0868 0 rpy=0 0 0
